File: hardware/LocalTrack.kicad_sch (KiCad schematic)
At the start: 59 parts, among them CON1 ST-LINK_V2, J1 USB_B_Micro, Q1 SI2302, Q2 SI2302, Q3 SI2302, Q4 SI2301, Q5 SI2302, Q6 SI2301, SW1 KCD1-11, U1 ADXL345BCCZ, U2 IP4220CZ6, U3 STM32F072C8T6, U4 MCP73831T-2DCI, U5 MCP73831T-2DCI, U6 W25N01GVZEIG, U7 MCP1700T-3302E/TT, U9 SIM28, Y1 8MHz

Commit message: documentation update
Parts:
- SW1: value KCD1-11 -> KCD11-2P
- U4, U5: value MCP73831T-2DCI -> MCP73831T-2DCI/OT
Changed lines of the file:
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@@
     (in_bom yes) (on_board yes)
     (property "Reference" "U4" (id 0) (at 130.81 35.56 0))
-    (property "Value" "MCP73831T-2DCI" (id 1) (at 130.81 38.1 0))
+    (property "Value" "MCP73831T-2DCI/OT" (id 1) (at 130.81 38.1 0))
     (property "Footprint" "Package_TO_SOT_SMD:SOT-23-5" (id 2) (at 144.78 35.56 0)
       (effects (font (size 1.27 1.27) italic) (justify left) hide)
@@
     (in_bom yes) (on_board yes)
     (property "Reference" "SW1" (id 0) (at 232.41 16.891 0))
-    (property "Value" "KCD1-11" (id 1) (at 232.41 19.2024 0))
+    (property "Value" "KCD11-2P" (id 1) (at 232.41 19.2024 0))
     (property "Footprint" "LocalTrack:KCD1-11" (id 2) (at 232.41 22.86 0)
       (effects (font (size 1.27 1.27)) hide)
@@
     (in_bom yes) (on_board yes)
     (property "Reference" "U5" (id 0) (at 130.81 59.69 0))
-    (property "Value" "MCP73831T-2DCI" (id 1) (at 130.81 62.23 0))
+    (property "Value" "MCP73831T-2DCI/OT" (id 1) (at 130.81 62.23 0))
     (property "Footprint" "Package_TO_SOT_SMD:SOT-23-5" (id 2) (at 144.78 59.69 0)
       (effects (font (size 1.27 1.27) italic) (justify left) hide)
@@
     )
     (path "/00000000-0000-0000-0000-00005e750ce5"
-      (reference "SW1") (unit 1) (value "KCD1-11") (footprint "LocalTrack:KCD1-11")
+      (reference "SW1") (unit 1) (value "KCD11-2P") (footprint "LocalTrack:KCD1-11")
     )
     (path "/00000000-0000-0000-0000-00005f83d98d"
@@
     )
     (path "/00000000-0000-0000-0000-00005c7ee99f"
-      (reference "U4") (unit 1) (value "MCP73831T-2DCI") (footprint "Package_TO_SOT_SMD:SOT-23-5")
+      (reference "U4") (unit 1) (value "MCP73831T-2DCI/OT") (footprint "Package_TO_SOT_SMD:SOT-23-5")
     )
     (path "/00000000-0000-0000-0000-00005e7726b0"
-      (reference "U5") (unit 1) (value "MCP73831T-2DCI") (footprint "Package_TO_SOT_SMD:SOT-23-5")
+      (reference "U5") (unit 1) (value "MCP73831T-2DCI/OT") (footprint "Package_TO_SOT_SMD:SOT-23-5")
     )
     (path "/00000000-0000-0000-0000-00005e670d47"
